File: Hardware/Hardware.kicad_sch (KiCad schematic)
At the start: 0 parts

Commit message: Update SCH
Other:
- added sheet Ports (Ports.kicad_sch)
- sheet Brush_Motor ports: added C_Brush+, C_Brush-, L_Brush+, L_Brush-, R_Brush+, R_Brush-; removed none
Changed lines of the file:
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@@
+			)
+		)
+		(pin "C_Brush+" input
+			(at 144.78 69.85 0)
+			(effects
+				(font
+					(size 1.27 1.27)
+				)
+				(justify right)
+			)
+		)
+		(pin "C_Brush-" input
+			(at 144.78 72.39 0)
+			(effects
+				(font
+					(size 1.27 1.27)
+				)
+				(justify right)
+			)
+		)
+		(pin "R_Brush+" input
+			(at 144.78 76.2 0)
+			(effects
+				(font
+					(size 1.27 1.27)
+				)
+				(justify right)
+			)
+		)
+		(pin "R_Brush-" input
+			(at 144.78 78.74 0)
+			(effects
+				(font
+					(size 1.27 1.27)
+				)
+				(justify right)
+			)
+		)
+		(pin "L_Brush+" input
+			(at 144.78 82.55 0)
+			(effects
+				(font
+					(size 1.27 1.27)
+				)
+				(justify right)
+			)
+		)
+		(pin "L_Brush-" input
+			(at 144.78 85.09 0)
+			(effects
+				(font
+					(size 1.27 1.27)
+				)
+				(justify right)
 			)
 		)
@@
 	)
 	(sheet
+		(at 163.83 49.53)
+		(size 39.37 41.91)
+		(fields_autoplaced yes)
+		(stroke
+			(width 0.1524)
+			(type solid)
+		)
+		(fill
+			(color 0 0 0 0.0000)
+		)
+		(property "Sheetname" "Ports"
+			(at 163.83 48.8184 0)
+			(effects
+				(font
+					(size 1.27 1.27)
+				)
+				(justify left bottom)
+			)
+		)
+		(property "Sheetfile" "Ports.kicad_sch"
+			(at 163.83 92.0246 0)
+			(effects
+				(font
+					(size 1.27 1.27)
+				)
+				(justify left top)
+			)
+		)
+		(property "字段 2" ""
+			(at 163.83 49.53 0)
+			(effects
+				(font
+					(size 1.27 1.27)
+				)
+				(hide yes)
+			)
+		)
+		(pin "L_Wheel-" input
+			(at 163.83 58.42 180)
+			(effects
+				(font
+					(size 1.27 1.27)
+				)
+				(justify left)
+			)
+		)
+		(pin "L_Wheel+" input
+			(at 163.83 55.88 180)
+			(effects
+				(font
+					(size 1.27 1.27)
+				)
+				(justify left)
+			)
+		)
+		(pin "R_Wheel+" input
+			(at 163.83 63.5 180)
+			(effects
+				(font
+					(size 1.27 1.27)
+				)
+				(justify left)
+			)
+		)
+		(pin "R_Wheel-" input
+			(at 163.83 66.04 180)
+			(effects
+				(font
+					(size 1.27 1.27)
+				)
+				(justify left)
+			)
+		)
+		(instances
+			(project "Hardware"
+				(path "/8d39550c-1c23-48e1-ae23-c502e9088467"
+					(page "8")
+				)
+			)
+		)
+	)
+	(sheet
 		(at 90.17 15.24)
 		(size 20.32 26.67)
@@
 	)
 	(sheet
-		(at 179.07 40.64)
+		(at 119.38 161.29)
 		(size 39.37 64.77)
 		(fields_autoplaced yes)
@@
 		)
 		(property "Sheetname" "Sensors"
-			(at 179.07 39.9284 0)
+			(at 119.38 160.5784 0)
 			(effects
 				(font
@@
 		)
 		(property "Sheetfile" "Sensors.kicad_sch"
-			(at 179.07 105.9946 0)
-			(effects
-				(font
+			(at 119.38 226.6446 0)
+			(effects
+				(font

Commit message: Update PCB
Changed lines of the file:
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@@
 	)
 	(sheet
-		(at 119.38 161.29)
+		(at 143.51 102.87)
 		(size 39.37 64.77)
 		(fields_autoplaced yes)
@@
 		)
 		(property "Sheetname" "Sensors"
-			(at 119.38 160.5784 0)
+			(at 143.51 102.1584 0)
 			(effects
 				(font
@@
 		)
 		(property "Sheetfile" "Sensors.kicad_sch"
-			(at 119.38 226.6446 0)
+			(at 143.51 168.2246 0)
 			(effects
 				(font
