File: Hardware/IMU.kicad_sch (KiCad schematic)
At the start: 14 parts, among them Q1 AO3400

Commit message: Update PCB
Parts:
- removed C14, C16: 0.1uF, symbol Device:C
- removed C15: 1uF, symbol Device:C
- removed C17: 0.01uF, symbol Device:C
- removed Q1: AO3400, SOT95P280X125-3N, symbol SamacSys_Parts:AO3400
- removed R10, R12: 500R, symbol Device:R
- removed R11: IMU_Heater, SamacSys_Parts:IMU_Heater, symbol Device:R
- removed R5, R6, R7: 22R, symbol Device:R
- removed R8: 100R, symbol Device:R
- removed R9: 10K, symbol Device:R
- removed U2: ~, SamacSys_Parts:ICM20602, symbol SamacSys_Parts:ICM20602
Connections:
- no-connect marks 1 -> 0
