File: Hardware/Ports.kicad_sch (KiCad schematic)
At the start: 5 parts, among them J3 L_Wheel_Motor, J4 R_Wheel_Motor, J5 L_Brush_Motor, J6 R_Brush_Motor, J7 C_Brush_Motor

Commit message: Update PCB
Parts:
- added CN1: 2.54-2P_WT, kicad_lceda:CONN-SMD_2.54-2PWT, symbol Library:2.54-2P_WT
- added CN2: DF13B-2P-1.25V(51), kicad_lceda:CONN-TH_2P-P1.25_HRS_DF13B-2P-1.25V-51, symbol Library:DF13B-2P-1.25V(51)
- added CN3: UK-2.0-2AWT, kicad_lceda:CONN-SMD_2P-P2.00_USAKRO_UK-2.0-2AWT, symbol Library:UK-2.0-2AWT
- added CN4: UK-2.0-4AWT, kicad_lceda:CONN-SMD_4P-P2.00_USAKRO_UK-2.0-4AWT, symbol Library:UK-2.0-4AWT
- added J8: SMD1.25-6P, kicad_lceda:SMD-1.25-6P, symbol Library:SMD1.25-6P
- added J9: SMD1.25-8P, kicad_lceda:SMD-1.25-8P, symbol Library:SMD1.25-8P
- added P1: Header_6, kicad_lceda:CONN-SMD-6P-1.5, symbol Library:Header_6
- added U8: A1001WR-S-2X08PD01, kicad_lceda:CONN-SMD_A1001WR-S-2X08PD01, symbol Library:A1001WR-S-2X08PD01
- J3, J4, J5, J6, J7: symbol Connector:Conn_01x02_Socket -> Library:Conn_01x02_Socket
Connections:
- net C_Brush+: now reaches J7.1 (Pin_1)
- net C_Brush-: now reaches J7.2 (Pin_2)
- net R_Brush+: now reaches J6.1 (Pin_1)
- net R_Brush-: now reaches J6.2 (Pin_2)
- net L_Brush+: now reaches J5.1 (Pin_1)
- net L_Brush-: now reaches J5.2 (Pin_2)
Other:
- moved on the sheet: J3, J4, J5, J6, J7
