File: Hardware/Sensors.kicad_sch (KiCad schematic)
At the start: 14 parts, among them Q1 AO3400

Commit message: Add Image Transmission
Parts:
- removed C14, C16: 0.1uF, symbol Device:C
- removed C15: 1uF, symbol Device:C
- removed C17: 0.01uF, symbol Device:C
- removed Q1: AO3400, SOT95P280X125-3N, symbol SamacSys_Parts:AO3400
- removed R10, R12: 500R, symbol Device:R
- removed R11: IMU_Heater, SamacSys_Parts:IMU_Heater, symbol Device:R
- removed R5, R6, R7: 22R, symbol Device:R
- removed R8: 100R, symbol Device:R
- removed R9: 10K, symbol Device:R
- removed U2: ~, SamacSys_Parts:ICM20602, symbol SamacSys_Parts:ICM20602
Connections:
- no-connect marks 1 -> 0

Commit message: Update PCB
Parts:
- added C14, C16: 0.1uF, Capacitor_SMD:C_0603_1608Metric, symbol Library:C
- added C15: 1uF, Capacitor_SMD:C_0603_1608Metric, symbol Library:C
- added C17: 0.01uF, Capacitor_SMD:C_0603_1608Metric, symbol Library:C
- added Q1: AO3400, SOT95P280X125-3N, symbol Library:AO3400
- added R10, R12: 500R, Resistor_SMD:R_0603_1608Metric, symbol Library:R
- added R11: IMU_Heater, SamacSys_Parts:IMU_Heater, symbol Library:R
- added R5, R6, R7: 22R, Resistor_SMD:R_0603_1608Metric, symbol Library:R
- added R8: 100R, Resistor_SMD:R_0603_1608Metric, symbol Library:R
- added R9: 10K, Resistor_SMD:R_0603_1608Metric, symbol Library:R
- added U2: ~, SamacSys_Parts:ICM20602, symbol Library:ICM20602
Connections:
- new net: Q1.1 (G), R8.2, R9.2
- new net: R11.2, R12.1
- new net: Q1.3 (D), R12.2
- new net: R10.2, R11.1
- new net +3.3V: C17.2, U2.1 (VDDIO), U2.16 (VDD)
- new net GND: C14.1, C15.1, C16.2, C17.1, Q1.2 (S), R9.1, U2.10 (RESV), U2.11 (RESV), U2.12 (RESV), U2.13 (GND), U2.15 (RESV), U2.9 (RESV)
- new net IMU_CLK: R5.1, R5.2, U2.2 (SCL)
- new net IMU_CS: U2.5 (CS)
- new net IMU_FSYNC: U2.8 (FSYNC)
- new net IMU_Heater: R8.1
- new net IMU_INT: U2.6 (INT)
- new net IMU_MISO: R7.1, R7.2, U2.4 (AD0)
- new net IMU_MOSI: R6.1, R6.2, U2.3 (SDA)
- new net REGOUT: C16.1, U2.14 (REGOUT)
- new net VCC: R10.1
- new net VDD: C14.2, C15.2
- no-connect marks 0 -> 1
