File: Hardware/Wireless_Image_Transmission/Wireless_Image_Transmission.kicad_pcb (KiCad board)
At the start: 2 copper layers, 24.9 x 24.9 mm, 51 parts, among them IC1 W25Q32JVSSIQ, IC2 ESP32-D0WD, IC3 IPS6404L-SQ-SPN, J1 OV2640, Q1 AO3401A, U1 XC6206P282MR, U2 XC6206P122MR, Y1 YSX321SL_40Mhz

Commit message: Init PCB
Parts:
- moved C7 1.88 mm to (36.1, 71.3), turned to 0 degrees
- moved C9 1.56 mm to (34.6, 70.8), turned to 90 degrees
- moved C18 1.49 mm to (36.5, 66.9), turned to -90 degrees
- moved R4 1.36 mm to (41.8, 82.3)
- moved C10 1.06 mm to (39.0, 66.4)
- moved C11 1.03 mm to (37.5, 66.9)
- moved L2 1.00 mm to (35.5, 68.8)
- moved C8 1.00 mm to (39.0, 67.4)
- moved C5 0.96 mm to (36.5, 68.8)
- moved C1 0.96 mm to (38.4, 68.8)
- moved C2 0.95 mm to (37.5, 68.8)
- moved C15 0.94 mm to (39.4, 68.8)
- moved C19 0.89 mm to (38.0, 70.3)
- moved C20 0.88 mm to (39.4, 70.7)
- moved C22 0.88 mm to (36.1, 70.3), turned to 180 degrees
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Routing:
- net /CSI_HSYNC: track 0.00 -> 26.2 mm, vias 0 -> 2
- net /CSI_D0: track 0.00 -> 20.6 mm, vias 0 -> 2
- net +3.3V: track 0.00 -> 19.5 mm, vias 0 -> 2
- net /CSI_D1: track 0.00 -> 16.3 mm, vias 0 -> 2
- net /CSI_D3: track 0.00 -> 15.2 mm
- net /CSI_D2: track 0.00 -> 13.8 mm
- net +3.3VADC: track 0.00 -> 11.7 mm, vias 0 -> 1
- net /XTAL_N: track 0.00 -> 4.66 mm
- net /CAP1: track 0.00 -> 4.25 mm, vias 0 -> 1
- net /CAP2: track 0.00 -> 3.87 mm, vias 0 -> 1
- net /CSI_D4: track 0.00 -> 3.39 mm
- net /XTAL_P: track 0.00 -> 2.81 mm
- net /CAM_RST: track 0.00 -> 2.20 mm
- net /TWI_SCL: track 0.00 -> 1.93 mm
- net /TWI_SDA: track 0.00 -> 1.83 mm
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- added copper zone on B.Cu, net GND
- added copper zone on F.Cu, net GND

Commit message: Update PCB
Parts:
- added ?: , SamacSys_Parts:nya_mini, F.Cu at (49.2, 70.4)
- added JP1: EN, Jumper:SolderJumper-2_P1.3mm_Open_RoundedPad1.0x1.5mm, F.Cu at (26.1, 87.7)
- moved R10 10.0 mm to (27.5, 82.2), turned to 0 degrees
- moved C29 7.60 mm to (29.4, 82.2), turned to 180 degrees
- moved C17 4.98 mm to (26.8, 64.3)
- moved C3 3.53 mm to (45.6, 68.1), turned to 90 degrees
- moved C6 2.24 mm to (43.9, 67.6), turned to 180 degrees
- moved L1 1.19 mm to (43.9, 68.6), turned to 180 degrees
- moved R3 0.70 mm to (41.3, 82.3)
- moved C23 0.70 mm to (40.2, 82.3)
- moved R7 0.56 mm to (39.1, 82.3)
- moved R4 0.55 mm to (42.4, 82.3)
- moved R9 0.42 mm to (38.1, 82.3)
- moved C25 0.29 mm to (37.0, 82.3)
- moved C21 0.28 mm to (41.8, 65.6)
- moved R5 0.25 mm to (41.8, 66.6)
- moved C13 0.24 mm to (41.8, 68.6)
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Connections:
- C27 pad 1: CSI-1.8V -> CSI_2.8V
- C30 pad 1: CSI-1.8V -> CSI_1.8V
- IC3 pad 1: /PSRAM_CLK -> /PSRAM_CS
- J1 pad 15: CSI-1.8V -> CSI_1.8V
- R10 pad 2: /PSRAM_CLK -> /PSRAM_CS
- U1 pad 2: CSI-1.8V -> CSI_2.8V
- U2 pad 2: CSI-1.8V -> CSI_1.8V
Routing:
- net +3.3V: track 19.5 -> 82.5 mm, vias 2 -> 10
- net /CSI_MCLK: track 0.00 -> 40.0 mm, vias 0 -> 5
- net /CSI_D7: track 0.00 -> 36.6 mm, vias 0 -> 6
- net /SDIO_D1: track 0.00 -> 34.4 mm
- net /CSI_D6: track 0.00 -> 33.5 mm, vias 0 -> 6
- net /CSI_D5: track 0.00 -> 31.6 mm, vias 0 -> 4
- net /CSI_VSYNC: track 0.00 -> 30.4 mm, vias 0 -> 2
- net /SDIO_D2: track 0.00 -> 30.4 mm
- net /TWI_SCL: track 1.93 -> 30.5 mm, vias 0 -> 2
- net /CSI_D4: track 3.39 -> 31.2 mm, vias 0 -> 6
- net /TWI_SDA: track 1.83 -> 28.8 mm, vias 0 -> 2
- net /PSRAM_CS: track 0.00 -> 22.1 mm, vias 0 -> 4
- net /U0TXD: track 0.00 -> 20.8 mm, vias 0 -> 2
- net /CSI_PCLK: track 0.00 -> 19.1 mm, vias 0 -> 2
- net /CAM_PWR: track 0.00 -> 18.8 mm, vias 0 -> 2
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- added copper zone on B.Cu, net +3.3V
- added copper zone on B.Cu, net /U0RXD
- added copper zone on B.Cu, net /U0TXD
Other:
- board size 24.9 x 24.9 mm -> 27 x 27 mm
- board text added: "0"
- board text added: "0 mm"
- board text added: "0.01 mm"
- board text added: "0.02"
- board text added: "0.035 mm"
- board text added: "1"
- board text added: "1.51 mm"
- board text added: "3.3"
- board text added: "4.5"
- board text added: "B.Cu"
- board text added: "B.Mask"
- board text added: "B.Paste"
- board text added: "B.Silkscreen"
- board text added: "Bottom Silk Screen"
- board text added: "Bottom Solder Mask"
- board text added: "Bottom Solder Paste"
- board text added: "Epsilon R"
- board text added: "F.Cu"
- board text added: "F.Mask"
- board text added: "F.Paste"
- board text added: "F.Silkscreen"
- board text added: "FR4"
- board text added: "Loss Tangent"
- board text added: "Not specified"
- board text added: "Top Silk Screen"
- board text added: "Top Solder Mask"
- board text added: "Top Solder Paste"
- board text added: "copper"
- board text added: "core"
- board text added: "介质 1"
- board text added: "厚度 (mm)"
- board text added: "层名称"
- board text added: "材料"
- board text added: "类型"
- board text added: "颜色"
